File: board/main/main.brd (EAGLE design)
At the start: 123.6 x 35.4 mm, 35 parts, among them IC1 78m05, J1 188275-8, U1 6N138M, U2 MMBD4148TW-7-F, U3 MMBD4148TW-7-F, U4 MMBD4148TW-7-F, U5 BAT54SDW-7-F

Commit message: Improving trigger responses (#2)
Parts:
- removed R5, R8: 100, SparkFun-Resistors:1206
- RN2: value 2.2K -> 10K
- moved R4 24.7 mm to (66.2, 33.0), turned to 180 degrees
- moved C6 19.4 mm to (87.7, 21.0), turned to 90 degrees
- moved U1 17.3 mm to (67.6, 25.7), turned to 0 degrees
- moved R6 12.2 mm to (14.7, 5.69)
- moved R7 12.0 mm to (76.9, 22.1), turned to 0 degrees
- moved R3 11.9 mm to (76.9, 18.9), turned to 0 degrees
- moved J1 9.80 mm to (85.6, 33.0)
- moved R1 9.00 mm to (66.4, 18.2)
- moved RN3 5.61 mm to (113.3, 30.4), turned to 0 degrees
- moved RN2 5.20 mm to (108.0, 32.0)
- moved RN1 5.16 mm to (108.0, 29.0)
- moved U5 4.41 mm to (118.7, 30.3)
- moved J2 1.41 mm to (83.4, 22.5)
Connections:
- net N$12 renamed J5-TIP
- net N$16 renamed J6-RING
- net N$2 renamed J3-TIP
- net N$9 renamed J4-RING
- removed net N$14: EXP.11, R5.1
- removed net N$18: EXP.12, RN3.1
- removed net N$19: EXP.5, R8.1
- removed net N$21: EXP.6, RN3.2
- net 3V: now also EXP.10, EXP.4; no longer R5.2, R8.2
- net AGND: now also RN3.7, RN3.8; no longer EXP.10, EXP.4
- net JACK1: now also EXP.6, RN3.1; no longer RN3.8
- net JACK2: now also EXP.12, RN3.2; no longer RN3.7
- net JACK3: now also RN1.7, RN2.6; no longer RN1.6, RN2.7
- net JACK4: now also RN1.5, RN2.8; no longer RN1.8, RN2.5
- net JACK5: now also RN1.6, RN2.7; no longer RN1.7, RN2.6
- net JACK6: now also RN1.8, RN2.5; no longer RN1.5, RN2.8
Routing:
- net AGND: track 187.0 -> 101.1 mm
- net N$19: track 21.6 -> 0.00 mm, vias 1 -> 0
- net JACK5: track 75.0 -> 96.4 mm
- net JACK6: track 97.3 -> 78.0 mm, vias 4 -> 3
- net N$14: track 18.0 -> 0.00 mm, vias 1 -> 0
- net 3V: track 99.1 -> 115.7 mm, vias 1 -> 2
- net FS2_LED: track 34.5 -> 51.1 mm
- net N$21: track 16.4 -> 0.00 mm, vias 1 -> 0
- net TX: track 42.1 -> 26.4 mm
- net VIN: track 98.8 -> 113.0 mm, vias 1 -> 2
- net ACT_LED: track 23.4 -> 36.3 mm
- net N$18: track 10.9 -> 0.00 mm
- net SIG-A: track 64.2 -> 53.8 mm, vias 3 -> 1
- net FS2: track 27.0 -> 36.8 mm
- net FS3: track 26.9 -> 36.7 mm
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- added copper zone on layer 16, net AGND
Other:
- board text added: "12/24/2020 REV: F"
- board text removed: "11/15/2020 REV: E"
