File: board/main/main.sch (EAGLE design)
At the start: 35 parts, among them IC1 78m05, J1 188275-8, U1 6N138M, U2 MMBD4148TW-7-F, U3 MMBD4148TW-7-F, U4 MMBD4148TW-7-F, U5 BAT54SDW-7-F

Commit message: Improving trigger responses (#2)
Parts:
- removed R5, R8: 100, SparkFun-Resistors:RESISTOR1206
- RN2: value 2.2K -> 10K
Connections:
- net N$12 renamed J5-TIP
- net N$16 renamed J6-RING
- net N$2 renamed J3-TIP
- net N$9 renamed J4-RING
- removed net N$14: EXP.P$11, R5.1
- removed net N$18: EXP.P$12, RN3A.1
- removed net N$19: EXP.P$5, R8.1
- removed net N$21: EXP.P$6, RN3B.1
- net 3V: now also EXP.P$10, EXP.P$4; no longer R5.2, R8.2
- net AGND: now also RN3A.2, RN3B.2; no longer EXP.P$10, EXP.P$4
- net JACK1: now also EXP.P$6, RN3A.1; no longer RN3A.2
- net JACK2: now also EXP.P$12, RN3B.1; no longer RN3B.2
- net JACK3: now also RN1B.2, RN2C.2; no longer RN1C.2, RN2B.2
- net JACK4: now also RN1D.2, RN2A.2; no longer RN1A.2, RN2D.2
- net JACK5: now also RN1C.2, RN2B.2; no longer RN1B.2, RN2C.2
- net JACK6: now also RN1A.2, RN2D.2; no longer RN1D.2, RN2A.2
